Commit message: First commit

File: legged_examples/legged_hunter/legged_hunter_description/urdf/hunter.urdf (robot description, URDF)
Before this commit: robot hunter, 16 links, 15 joints
Links:
- link leg_l5_link: geometry collision box size=0.1501 0.0345 0.0175; visual mesh filename=package://legged_hunter_description/meshes/leg_l5_link.STL
- link leg_r5_link: geometry collision box size=0.1501 0.0345 0.0175; visual mesh filename=package://legged_hunter_description/meshes/leg_r5_link.STL
Joints:
- joint leg_l4_joint: origin xyz=0 0.0145 -0.24 rpy=0 0 0 -> xyz=0 0.0145 -0.344 rpy=0 0 0
- joint leg_l5_joint: origin xyz=0.005 0 -0.23995 rpy=0 0 0 -> xyz=0.005 0 -0.344 rpy=0 0 0
- joint leg_r4_joint: origin xyz=0 -0.0145 -0.24 rpy=0 0 0 -> xyz=0 -0.0145 -0.344 rpy=0 0 0
- joint leg_r5_joint: origin xyz=0.005 0 -0.23995 rpy=0 0 0 -> xyz=0.005 0 -0.344 rpy=0 0 0

File: legged_examples/legged_hunter/legged_hunter_description/urdf/hunter_sim.urdf (robot description, URDF)
Before this commit: robot hunter, 16 links, 15 joints
Links:
- link leg_l5_link: geometry collision box size=0.1501 0.0345 0.0175; visual mesh filename=package://legged_hunter_description/meshes/leg_l5_link.STL
- link leg_r5_link: geometry collision box size=0.1501 0.0345 0.0175; visual mesh filename=package://legged_hunter_description/meshes/leg_r5_link.STL
Joints:
- joint leg_l4_joint: origin xyz=0 0.0145 -0.24 rpy=0 0 0 -> xyz=0 0.0145 -0.344 rpy=0 0 0
- joint leg_l5_joint: origin xyz=0.005 0 -0.23995 rpy=0 0 0 -> xyz=0.005 0 -0.344 rpy=0 0 0
- joint leg_r4_joint: origin xyz=0 -0.0145 -0.24 rpy=0 0 0 -> xyz=0 -0.0145 -0.344 rpy=0 0 0
- joint leg_r5_joint: origin xyz=0.005 0 -0.23995 rpy=0 0 0 -> xyz=0.005 0 -0.344 rpy=0 0 0

Commit message: Replaced Leg lengths and hip width with exo specs

File: legged_examples/legged_hunter/legged_hunter_description/urdf/hunter.urdf (robot description, URDF)
Before this commit: robot hunter, 16 links, 15 joints
Links:
- link leg_l5_link: geometry collision box size=0.2301 0.0345 0.0175; visual mesh filename=package://legged_hunter_description/meshes/leg_l5_link.STL
- link leg_r5_link: geometry collision box size=0.2301 0.0345 0.0175; visual mesh filename=package://legged_hunter_description/meshes/leg_r5_link.STL
Joints:
- joint leg_l1_joint: origin xyz=-0.002 0.09 -0.1035 rpy=0 0 0 -> xyz=-0.002 0.175 -0.1035 rpy=0 0 0
- joint leg_l4_joint: origin xyz=0 0.0145 -0.344 rpy=0 0 0 -> xyz=0 0.0145 -0.468 rpy=0 0 0
- joint leg_l5_fixed_1: origin xyz=0.06 0 -0.007 rpy=0 0 0 -> xyz=0.12 0 -0.007 rpy=0 0 0
- joint leg_l5_fixed_2: origin xyz=-0.030 0 -0.007 rpy=0 0 0 -> xyz=-0.090 0 -0.007 rpy=0 0 0
- joint leg_l5_joint: origin xyz=0.005 0 -0.344 rpy=0 0 0 -> xyz=0.005 0 -0.468 rpy=0 0 0
- joint leg_r1_joint: origin xyz=-0.002 -0.09 -0.1035 rpy=0 0 0 -> xyz=-0.002 -0.175 -0.1035 rpy=0 0 0
- joint leg_r4_joint: origin xyz=0 -0.0145 -0.344 rpy=0 0 0 -> xyz=0 -0.0145 -0.468 rpy=0 0 0
- joint leg_r5_fixed_1: origin xyz=0.06 0 -0.007 rpy=0 0 0 -> xyz=0.12 0 -0.007 rpy=0 0 0
- joint leg_r5_fixed_2: origin xyz=-0.030 0 -0.007 rpy=0 0 0 -> xyz=-0.090 0 -0.007 rpy=0 0 0
- joint leg_r5_joint: origin xyz=0.005 0 -0.344 rpy=0 0 0 -> xyz=0.005 0 -0.468 rpy=0 0 0

File: legged_examples/legged_hunter/legged_hunter_description/urdf/hunter_sim.urdf (robot description, URDF)
Before this commit: robot hunter, 16 links, 15 joints
Links:
- link leg_l5_link: geometry collision box size=0.2301 0.0345 0.0175; visual mesh filename=package://legged_hunter_description/meshes/leg_l5_link.STL
- link leg_r5_link: geometry collision box size=0.2301 0.0345 0.0175; visual mesh filename=package://legged_hunter_description/meshes/leg_r5_link.STL
Joints:
- joint leg_l1_joint: origin xyz=-0.002 0.09 -0.1035 rpy=0 0 0 -> xyz=-0.002 0.175 -0.1035 rpy=0 0 0
- joint leg_l4_joint: origin xyz=0 0.0145 -0.344 rpy=0 0 0 -> xyz=0 0.0145 -0.468 rpy=0 0 0
- joint leg_l5_fixed_1: origin xyz=0.06 0 -0.007 rpy=0 0 0 -> xyz=0.12 0 -0.007 rpy=0 0 0
- joint leg_l5_fixed_2: origin xyz=-0.030 0 -0.007 rpy=0 0 0 -> xyz=-0.090 0 -0.007 rpy=0 0 0
- joint leg_l5_joint: origin xyz=0.005 0 -0.344 rpy=0 0 0 -> xyz=0.005 0 -0.468 rpy=0 0 0
- joint leg_r1_joint: origin xyz=-0.002 -0.09 -0.1035 rpy=0 0 0 -> xyz=-0.002 -0.175 -0.1035 rpy=0 0 0
- joint leg_r4_joint: origin xyz=0 -0.0145 -0.344 rpy=0 0 0 -> xyz=0 -0.0145 -0.468 rpy=0 0 0
- joint leg_r5_fixed_1: origin xyz=0.06 0 -0.007 rpy=0 0 0 -> xyz=0.12 0 -0.007 rpy=0 0 0
- joint leg_r5_fixed_2: origin xyz=-0.030 0 -0.007 rpy=0 0 0 -> xyz=-0.090 0 -0.007 rpy=0 0 0
- joint leg_r5_joint: origin xyz=0.005 0 -0.344 rpy=0 0 0 -> xyz=0.005 0 -0.468 rpy=0 0 0
